Commit message: 备份：清洁机器人工程阶段更新

File: src/cleanrobot_description/urdf/a26022_clean_robot.urdf (robot description, URDF)
Before this commit: robot a26022_clean_robot, 6 links, 5 joints
Links:
- added link gemini_cf_link
- added link gemini_front_link
- added link gemini_nj_link
- added link left_camera, mass 0.046; collision mesh filename=package://cleanrobot_description/meshes/left_camera.STL; visual mesh filename=package://cleanrobot_description/meshes/left_camera.STL
- added link right_camera, mass 0.046; collision mesh filename=package://cleanrobot_description/meshes/right_camera.STL; visual mesh filename=package://cleanrobot_description/meshes/right_camera.STL
- added link up_camera, mass 0.17239; collision mesh filename=package://cleanrobot_description/meshes/up_camera.STL; visual mesh filename=package://cleanrobot_description/meshes/up_camera.STL
Joints:
- added joint gemini_cf_mount: type fixed, parent base_link, child gemini_cf_link, origin xyz=-0.13292 0.32478 0.910841616448 rpy=-1.10771564304 0.70386486547 0.807282164799
- added joint gemini_front_mount: type fixed, parent base_link, child gemini_front_link, origin xyz=0.57945 0 0.97641 rpy=0.0038898 0.8874465 0
- added joint gemini_nj_mount: type fixed, parent base_link, child gemini_nj_link, origin xyz=-0.13292 -0.32478 0.949244255794 rpy=1.10708972437 0.665196470572 -0.814678120843
- added joint left_camera_joint: type fixed, parent base_link, child left_camera, origin xyz=-0.13292 0.32478 0.8656 rpy=0 0 0, axis 0 0 0
- added joint right_camera_joint: type fixed, parent base_link, child right_camera, origin xyz=-0.13292 -0.32478 0.8656 rpy=0 0 0, axis 0 0 0
- added joint up_camera_joint: type fixed, parent base_link, child up_camera, origin xyz=0.57945 0 0.97641 rpy=0 0 0, axis 0 0 0

Commit message: release: optimize coverage and global paths, repair MPPI control
优化了全覆盖路径  全局路径 修复了mppi运动控制算法

File: src/cleanrobot_description/urdf/a26022_clean_robot.urdf (robot description, URDF)
Before this commit: robot a26022_clean_robot, 12 links, 11 joints
Joints:
- joint gemini_cf_mount: origin xyz=-0.13292 0.32478 0.910841616448 rpy=-1.10771564304 0.70386486547 0.807282164799 -> xyz=-0.13292 0.32478 0.834894653381 rpy=-1.01965089 0.78006446 0.86685493
- joint gemini_nj_mount: origin xyz=-0.13292 -0.32478 0.949244255794 rpy=1.10708972437 0.665196470572 -0.814678120843 -> xyz=-0.13292 -0.32478 0.882211096476 rpy=1.04693284 0.70714258 -0.84837366
